File: Schematic & PCB/USB-C-12V-2A-BUCK-BOOST-CONVERTER/USB-C-12V-2A-BUCK-BOOST-CONVERTER.kicad_pcb (KiCad board)
At the start: 2 copper layers, 23 parts, among them J1 Conn_01x02_Pin, U1 TPS61089RNRR

Commit message: Added Gerber, BOM, and Pos
Parts:
- C9: footprint Capacitor_SMD:C_0603_1608Metric -> Capacitor_SMD:C_0805_2012Metric
- moved R2 44.7 mm to (132.1, 96.5), turned to -90 degrees
- moved R1 42.2 mm to (132.1, 82.5), turned to 90 degrees
- moved R3 23.4 mm to (162.6, 86.4), turned to -90 degrees
- moved R6 22.9 mm to (157.5, 86.4), turned to -90 degrees
- moved R5 22.0 mm to (160.0, 86.4), turned to 90 degrees
- moved R7 20.0 mm to (158.1, 78.7)
- moved C7 13.6 mm to (166.9, 85.4)
- moved C8 13.0 mm to (166.9, 87.2)
- moved J1 12.9 mm to (177.8, 83.8)
- moved C9 8.65 mm to (161.3, 82.2), turned to -90 degrees
- moved C1 8.28 mm to (156.8, 76.8), turned to 0 degrees
- moved C12 8.07 mm to (171.4, 82.2), turned to -90 degrees
- moved C11 5.15 mm to (168.3, 82.2), turned to -90 degrees
- moved C10 5.13 mm to (165.1, 82.2), turned to -90 degrees
- moved C2 0.95 mm to (150.2, 91.4)
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Routing:
- net Net-(U1-EN): track 0.00 -> 15.8 mm, vias 0 -> 2
- net Net-(U1-COMP): track 0.00 -> 10.7 mm
- net Net-(J1-Pin_2): track 0.00 -> 7.43 mm, vias 0 -> 2
- net Net-(USB1-CC1): track 0.00 -> 7.06 mm
- net Net-(USB1-CC2): track 0.00 -> 6.99 mm
- net Net-(U1-FB): track 0.00 -> 4.75 mm
- net VBUS: track 0.00 -> 4.56 mm
- net Net-(U1-FSW): track 0.00 -> 4.55 mm
- net Net-(C8-Pad1): track 0.00 -> 3.61 mm
- net Net-(U1-BOOT): track 0.00 -> 3.52 mm
- net Net-(U1-ILIM): track 0.00 -> 2.95 mm
- net GND: vias 0 -> 58
- added copper zone on B.Cu, net GND
- added copper zone on F.Cu, net GND
- added copper zone on F.Cu, net Net-(J1-Pin_2)
- added copper zone on F.Cu, net Net-(U1-SW)
- added copper zone on F.Cu, net VBUS
Other:
- board outline added: 55.2 x 26.7 mm
- board text added: "12V"
- board text added: "GND"
- board text added: "Victor Rosales USB-C to 12V Switching Boost Converter 12V-2A @24W MAX"
