File: Schematic & PCB REV 2/USB-C-12V-2A-BUCK-BOOST-CONVERTER/USB-C-12V-2A-BUCK-BOOST-CONVERTER.kicad_pcb (KiCad board)
At the start: 2 copper layers, 55.2 x 26.7 mm, 23 parts, among them J1 Conn_01x02_Pin, U1 TPS61089RNRR

Commit message: Final pcb review
Parts:
- removed the R1 at (132.1, 82.5)
- removed the R2 at (132.1, 96.5)
- removed USB1: USB4125-GF-A, lcsc_footprints:C3151650_USB-C-SMD_TYPE-C-6P
- added 5V: LED, lcsc_footprints:C84256_LED0805-RD, F.Cu at (135.3, 80.6)
- added 9V: 0805, lcsc_footprints:C2297_LED0805-R-RD, F.Cu at (135.1, 96.0)
- added C13: 100nF, Capacitor_SMD:C_0603_1608Metric, F.Cu at (149.9, 91.4)
- added PD: CH224K, lcsc_footprints:C970725_ESSOP-10_L4_9-W3_9-P1_0-LS6_0-TL-EP, F.Cu at (142.3, 94.2)
- added R10: 10k-0805, Resistor_SMD:R_0805_2012Metric, F.Cu at (143.3, 99.1)
- added R6: 4.7k-0805, Resistor_SMD:R_0805_2012Metric, F.Cu at (135.1, 82.8)
- added R7: 1k-0805, Resistor_SMD:R_0805_2012Metric, F.Cu at (146.3, 90.9)
- added R8: 6.8k-0805, Resistor_SMD:R_0805_2012Metric, F.Cu at (150.2, 99.6)
- added R9: 3.3k-0805, Resistor_SMD:R_0805_2012Metric, F.Cu at (135.1, 98.6)
- added USB-C: GT-USB-7010ASV, lcsc_footprints:C2988369_USB-C-SMD_G-SWITCH_GT-USB-7010ASV, F.Cu at (134.0, 89.5)
- moved L1 3.31 mm to (146.8, 84.8)
- moved C2 2.03 mm to (150.2, 93.5)
- moved C3 0.89 mm to (150.2, 95.5)
- moved C4 0.25 mm to (150.2, 97.5)
- renumbered C7 to C6, C8 to C7, C6 to C8, R3 to R1, R7 to R2, R4 to R3, R5 to R4, R6 to R5, U1 to U3
Routing:
- net CC1: track 0.00 -> 16.0 mm, vias 0 -> 2
- net DP: track 0.00 -> 13.4 mm, vias 0 -> 3
- net CC2: track 0.00 -> 12.8 mm, vias 0 -> 2
- net Net-(LED2-K): track 0.00 -> 12.4 mm, vias 0 -> 2
- net GND: track 0.00 -> 10.7 mm, vias 58 -> 60
- net DM: track 0.00 -> 9.97 mm, vias 0 -> 3
- net VDD: track 0.00 -> 9.84 mm, vias 0 -> 2
- net Net-(U2-CFG1): track 0.00 -> 9.45 mm, vias 0 -> 2
- net Net-(USB1-CC1): track 7.06 -> 0.00 mm
- net Net-(USB1-CC2): track 6.99 -> 0.00 mm
- net Net-(LED1-+): track 0.00 -> 3.05 mm
- net Net-(LED2-A): track 0.00 -> 2.60 mm
- net Net-(U2-VBUS): track 0.00 -> 1.91 mm

Commit message: Rev finished board
Parts:
- renumbered USB-C to U1, PD to U2
Connections:
- net Net-(J1-Pin_2) renamed +12V
Routing:
- net VDD: track 9.84 -> 27.9 mm, vias 2 -> 4
- net DP: track 13.4 -> 10.2 mm, vias 3 -> 2
- net GND: track 10.7 -> 12.8 mm, vias 60 -> 61
- net DM: track 9.97 -> 8.93 mm, vias 3 -> 2
Other:
- board size 55.2 x 26.7 mm -> 54.4 x 27.9 mm
